Commit message: Removed some stuff from hyq urdf to provide 16.04 compatibility

File: ct_models/urdf/HyQ/hyqb.urdf.xacro (robot description, xacro)
@@ -18,5 +18,5 @@
 	<!-- trunk -->
 	<xacro:hyq_trunk name="base">
-		<origin xyz="-0.443 -0.191 -0.276" rpy="0 0 0"/>
+		<!-- <origin xyz="-0.443 -0.191 -0.276" rpy="0 0 0"/> -->
 	</xacro:hyq_trunk>
 	<!-- LF leg -->
@@ -56,4 +56,3 @@
 		<origin xyz="${-d_fh/2} ${-d_lr/2} 0" rpy="0 ${PI/2} 0"/>
 	</xacro:hyq_leg>
--->
 </robot>

File: ct_models/urdf/HyQ/links/trunk.urdf.xacro (robot description, xacro)
@@ -39,5 +39,5 @@
 		</link>
 		<!-- Extensions -->
-		<xacro:trunk_gazebo name="trunk"/>
+		<!-- <xacro:trunk_gazebo name="trunk"/> -->
 	</xacro:macro>
 </robot>
