Commit message: making mesh files for quadrotor and quadrotor with load unique

File: ct_models/urdf/QuadrotorWithLoad/ct_quadrotor.urdf (robot description, URDF)
Before this commit: robot ct_quadrotor, 4 links, 3 joints
Links:
- link body: geometry visual mesh filename=package://ct_models/urdf/Quadrotor/quadrotor_base.dae scale=0.1 0.1 0.1
