Commit message: updating ct_models inverted pendulum the paramters of real pendulum

File: ct_models/urdf/InvertedPendulum/InvertedPendulum.urdf (robot description, URDF)
Before this commit: robot InvertedPendulum, 2 links, 1 joints
Links:
- link InvertedPendulumBase: geometry visual cylinder length=0.015 radius=0.015
- link Link1: mass 1.0 -> 1.811; geometry visual cylinder length=0.27 radius=0.01
